File: _autosave-16Bars.kicad_pcb (KiCad board)
At the start: 2 copper layers, 30 x 69 mm, 17 parts, among them IC1 CD4033BE, IC2 CD4033BE, J1 CLOCK_IN, J2 Conn_02x05_Odd_Even, SW1 RESET

Commit message: Let there be bars
Parts:
- moved SW1 42.3 mm to (76.2, 132.2)
- moved J1 36.5 mm to (61.5, 137.8)
Other:
- board size 30 x 69 mm -> 30 x 105 mm
Changed lines of the file:
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@@
   )
   (footprint "Connector_Audio:Jack_3.5mm_QingPu_WQP-PJ398SM_Vertical_CircularHoles" (layer "F.Cu")
-    (at 61.5 101.28 180)
+    (at 61.5 137.78 180)
     (descr "TRS 3.5mm, vertical, Thonkiconn, PCB mount, (http://www.qingpu-electronics.com/en/products/WQP-PJ398SM-362.html)")
     (tags "WQP-PJ398SM WQP-PJ301M-12 TRS 3.5mm mono vertical jack thonkiconn qingpu")
@@
   )
   (footprint "Button_Switch_THT:SW_PUSH_6mm" (layer "F.Cu")
-    (at 75 90)
+    (at 76.25 132.25)
     (descr "https://www.omron.com/ecb/products/pdf/en-b3f.pdf")
     (tags "tact sw push 6mm")
@@
     )
   )
-  (gr_line locked (start 55 35) (end 55 104) (layer "Edge.Cuts") (width 0.1))
-  (gr_line locked (start 55 104) (end 85 104) (layer "Edge.Cuts") (width 0.1))
+  (gr_line locked (start 55 140) (end 85 140) (layer "Edge.Cuts") (width 0.1))
   (gr_line locked (start 55 35) (end 85 35) (layer "Edge.Cuts") (width 0.1))
-  (gr_line locked (start 85 35) (end 85 104) (layer "Edge.Cuts") (width 0.1))
+  (gr_line locked (start 55 35) (end 55 140) (layer "Edge.Cuts") (width 0.1))
+  (gr_line locked (start 85 35) (end 85 140) (layer "Edge.Cuts") (width 0.1))
   (zone (net 6) (net_name "GND") (layer "B.Cu") (name "GroundPlane") (hatch edge 0.508)
     (connect_pads (clearance 0.508))
@@
     (polygon
       (pts
-        (xy 85 104)
-        (xy 55 104)
+        (xy 85 140)
+        (xy 55 140)
         (xy 55 35)
         (xy 85 35)
