File: _autosave-16Bars.kicad_sch (KiCad schematic)
At the start: 34 parts, among them IC1 CD4033BE, IC2 CD4033BE, IC3 CD4510BE, J1 CLOCK_IN, J2 Conn_02x05_Odd_Even, Q1 2N3904, Q2 2N3904, Q3 2N3904, Q4 2N3904, Q5 2N3904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

Commit message: Rough PCB Layout
Parts:
- renumbered DS-ONES to DS-ONES1, DS-TENS to DS-TENS1
Changed lines of the file:
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@@
   (symbol (lib_id "SamacSys_Parts:TDSR0760") (at 226.06 33.02 0) (unit 1)
     (in_bom yes) (on_board yes) (fields_autoplaced)
-    (property "Reference" "DS-ONES" (id 0) (at 242.57 25.4 0))
+    (property "Reference" "DS-ONES1" (id 0) (at 242.57 25.4 0))
     (property "Value" "TDSR0760" (id 1) (at 242.57 27.94 0))
     (property "Footprint" "SamacSys_Parts:TDSR0760" (id 2) (at 255.27 30.48 0)
@@
   (symbol (lib_id "SamacSys_Parts:TDSR0760") (at 226.06 73.66 0) (unit 1)
     (in_bom yes) (on_board yes) (fields_autoplaced)
-    (property "Reference" "DS-TENS" (id 0) (at 242.57 66.04 0))
+    (property "Reference" "DS-TENS1" (id 0) (at 242.57 66.04 0))
     (property "Value" "TDSR0760" (id 1) (at 242.57 68.58 0))
     (property "Footprint" "SamacSys_Parts:TDSR0760" (id 2) (at 255.27 71.12 0)
@@
     )
     (path "/273f01f0-28d2-4494-b80f-412095039d4d"
-      (reference "DS-ONES") (unit 1) (value "TDSR0760") (footprint "SamacSys_Parts:TDSR0760")
+      (reference "DS-ONES1") (unit 1) (value "TDSR0760") (footprint "SamacSys_Parts:TDSR0760")
     )
     (path "/d443e6a6-aeca-4918-a2c3-170714850785"
-      (reference "DS-TENS") (unit 1) (value "TDSR0760") (footprint "SamacSys_Parts:TDSR0760")
+      (reference "DS-TENS1") (unit 1) (value "TDSR0760") (footprint "SamacSys_Parts:TDSR0760")
     )
     (path "/fec73edc-3414-4808-9b3e-bbd5f70503c9"
