File: 16Bars.kicad_sch (KiCad schematic)
At the start: 34 parts, among them IC1 CD4033BE, IC2 CD4033BE, IC3 CD4510BE, J1 CLOCK_IN, J2 Conn_02x05_Odd_Even, Q1 2N3904, Q2 2N3904, Q3 2N3904, Q4 2N3904, Q5 2N3904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

Commit message: PCB Layout Complete
Parts:
- removed J1: CLOCK_IN, Connector_Audio:Jack_3.5mm_QingPu_WQP-PJ398SM_Vertical_CircularHoles, symbol eurocad:PJ301M-12
- added J1: CLOCK_IN, Connector_Audio:Jack_3.5mm_QingPu_WQP-PJ398SM_Vertical_CircularHoles, symbol Connector:AudioJack2
- R5: footprint Resistor_THT:R_Axial_DIN0207_L6.3mm_D2.5mm_P7.62mm_Horizontal -> Resistor_THT:R_Axial_DIN0204_L3.6mm_D1.6mm_P5.08mm_Horizontal
- R7: footprint Diode_THT:D_A-405_P7.62mm_Horizontal -> Resistor_THT:R_Axial_DIN0204_L3.6mm_D1.6mm_P5.08mm_Horizontal
- R8: footprint Resistor_SMD:R_0805_2012Metric -> Resistor_THT:R_Axial_DIN0204_L3.6mm_D1.6mm_P5.08mm_Horizontal
- renumbered DS-ONES to DS-ONES1, DS-TENS to DS-TENS1
Connections:
- net GND: now also J1.S; no longer IC2.14 (LAMPTEST)
- net at D1.2 (A): now also J1.T
Changed lines of the file:
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@@
   (no_connect (at 147.32 38.1))
   (no_connect (at 147.32 35.56))
-  (no_connect (at 154.94 138.43))
+  (no_connect (at 198.12 78.74))
   (no_connect (at 26.67 181.61))
   (no_connect (at 147.32 81.28))
@@
     (stroke (width 0) (type default) (color 0 0 0 0))
   )
-  (wire (pts (xy 156.21 134.62) (xy 154.94 134.62))
+  (wire (pts (xy 151.13 134.62) (xy 156.21 134.62))
     (stroke (width 0) (type default) (color 0 0 0 0))
   )
@@
     (stroke (width 0) (type default) (color 0 0 0 0))
   )
-  (wire (pts (xy 203.2 78.74) (xy 198.12 78.74))
-    (stroke (width 0) (type default) (color 0 0 0 0))
-  )
-  (wire (pts (xy 154.94 140.97) (xy 158.75 140.97))
-    (stroke (width 0) (type default) (color 0 0 0 0))
-  )
   (wire (pts (xy 265.43 78.74) (xy 259.08 78.74))
     (stroke (width 0) (type default) (color 0 0 0 0))
@@
     (stroke (width 0) (type default) (color 0 0 0 0))
   )
+  (wire (pts (xy 151.13 134.62) (xy 151.13 138.43))
+    (stroke (width 0) (type default) (color 0 0 0 0))
+  )
   (wire (pts (xy 110.49 38.1) (xy 114.3 38.1))
     (stroke (width 0) (type default) (color 0 0 0 0))
@@
   )
   (wire (pts (xy 147.32 48.26) (xy 147.32 55.88))
+    (stroke (width 0) (type default) (color 0 0 0 0))
+  )
+  (wire (pts (xy 151.13 140.97) (xy 158.75 140.97))
     (stroke (width 0) (type default) (color 0 0 0 0))
   )
@@
   (symbol (lib_id "SamacSys_Parts:TDSR0760") (at 226.06 33.02 0) (unit 1)
     (in_bom yes) (on_board yes) (fields_autoplaced)
-    (property "Reference" "DS-ONES" (id 0) (at 242.57 25.4 0))
+    (property "Reference" "DS-ONES1" (id 0) (at 242.57 25.4 0))
     (property "Value" "TDSR0760" (id 1) (at 242.57 27.94 0))
     (property "Footprint" "SamacSys_Parts:TDSR0760" (id 2) (at 255.27 30.48 0)
@@
     (pin "1")
   )
-  (symbol (lib_id "power:GND") (at 203.2 78.74 90) (unit 1)
-    (in_bom yes) (on_board yes)
-    (property "Reference" "#PWR021" (id 0) (at 209.55 78.74 0)
-      (effects (font (size 1.27 1.27)) hide)
-    )
-    (property "Value" "GND" (id 1) (at 207.01 81.28 0))
-    (property "Footprint" "" (id 2) (at 203.2 78.74 0)
-      (effects (font (size 1.27 1.27)) hide)
-    )
-    (property "Datasheet" "" (id 3) (at 203.2 78.74 0)
-      (effects (font (size 1.27 1.27)) hide)
-    )
-    (pin "1")
-  )
   (symbol (lib_id "Device:R") (at 41.91 92.71 90) (unit 1)
     (in_bom yes) (on_board yes) (fields_autoplaced)
@@
       (effects (font (size 1.27 1.27)) (justify right))
     )
-    (property "Footprint" "Diode_THT:D_A-405_P7.62mm_Horizontal" (id 2) (at 241.3 141.478 90)
+    (property "Footprint" "Resistor_THT:R_Axial_DIN0204_L3.6mm_D1.6mm_P5.08mm_Horizontal" (id 2) (at 241.3 141.478 90)
       (effects (font (size 1.27 1.27)) hide)
     )
@@
     (pin "2")
   )
+  (symbol (lib_id "Connector:AudioJack2") (at 146.05 140.97 0) (unit 1)
+    (in_bom yes) (on_board yes) (fields_autoplaced)
+    (property "Reference" "J1" (id 0) (at 145.415 132.08 0))
+    (property "Value" "CLOCK_IN" (id 1) (at 145.415 134.62 0))
+    (property "Footprint" "Connector_Audio:Jack_3.5mm_QingPu_WQP-PJ398SM_Vertical_CircularHoles" (id 2) (at 146.05 140.97 0)
+      (effects (font (size 1.27 1.27)) hide)
+    )
+    (property "Datasheet" "~" (id 3) (at 146.05 140.97 0)
+      (effects (font (size 1.27 1.27)) hide)
+    )
+    (pin "S")
+    (pin "T")
+  )
   (symbol (lib_id "power:GND") (at 186.69 59.69 270) (unit 1)
     (in_bom yes) (on_board yes)
@@
       (effects (font (size 1.27 1.27)) (justify left))
     )
-    (property "Footprint" "Resistor_SMD:R_0805_2012Metric" (id 2) (at 188.722 128.27 90)
+    (property "Footprint" "Resistor_THT:R_Axial_DIN0204_L3.6mm_D1.6mm_P5.08mm_Horizontal" (id 2) (at 188.722 128.27 90)
       (effects (font (size 1.27 1.27)) hide)
     )
@@
     (property "Reference" "R5" (id 0) (at 175.26 138.43 90))
     (property "Value" "47K" (id 1) (at 175.26 140.97 90))
-    (property "Footprint" "Resistor_THT:R_Axial_DIN0207_L6.3mm_D2.5mm_P7.62mm_Horizontal" (id 2) (at 175.26 139.192 90)
+    (property "Footprint" "Resistor_THT:R_Axial_DIN0204_L3.6mm_D1.6mm_P5.08mm_Horizontal" (id 2) (at 175.26 139.192 90)
       (effects (font (size 1.27 1.27)) hide)
     )
@@
   (symbol (lib_id "SamacSys_Parts:TDSR0760") (at 226.06 73.66 0) (unit 1)
     (in_bom yes) (on_board yes) (fields_autoplaced)
-    (property "Reference" "DS-TENS" (id 0) (at 242.57 66.04 0))
+    (property "Reference" "DS-TENS1" (id 0) (at 242.57 66.04 0))
     (property "Value" "TDSR0760" (id 1) (at 242.57 68.58 0))
     (property "Footprint" "SamacSys_Parts:TDSR0760" (id 2) (at 255.27 71.12 0)
@@
     (pin "2")
   )
-  (symbol (lib_id "eurocad:PJ301M-12") (at 143.51 138.43 0) (unit 1)
-    (in_bom yes) (on_board yes)
-    (property "Reference" "J1" (id 0) (at 143.6624 128.905 0))
-    (property "Value" "CLOCK_IN" (id 1) (at 143.6624 131.2164 0))
-    (property "Footprint" "Connector_Audio:Jack_3.5mm_QingPu_WQP-PJ398SM_Vertical_CircularHoles" (id 2) (at 143.51 138.43 0)
-      (effects (font (size 1.27 1.27)) hide)
-    )
-    (property "Datasheet" "" (id 3) (at 143.51 138.43 0))
-    (pin "1")
-    (pin "2")
-    (pin "3")
-  )
   (symbol (lib_id "power:GND") (at 49.53 26.67 270) (unit 1)
     (in_bom yes) (on_board yes)
@@
       (reference "#PWR020") (unit 1) (value "GND") (footprint "")
     )
-    (path "/3536541e-242a-48ec-ac08-b3ed00b9bd5f"
-      (reference "#PWR021") (unit 1) (value "GND") (footprint "")
-    )
     (path "/ceb92170-1ec5-43a6-addc-5b9134f6a428"
       (reference "#PWR022") (unit 1) (value "GND") (footprint "")
@@
     )
     (path "/273f01f0-28d2-4494-b80f-412095039d4d"
-      (reference "DS-ONES") (unit 1) (value "TDSR0760") (footprint "SamacSys_Parts:TDSR0760")
+      (reference "DS-ONES1") (unit 1) (value "TDSR0760") (footprint "SamacSys_Parts:TDSR0760")
     )
     (path "/d443e6a6-aeca-4918-a2c3-170714850785"
-      (reference "DS-TENS") (unit 1) (value "TDSR0760") (footprint "SamacSys_Parts:TDSR0760")
+      (reference "DS-TENS1") (unit 1) (value "TDSR0760") (footprint "SamacSys_Parts:TDSR0760")
     )
     (path "/fec73edc-3414-4808-9b3e-bbd5f70503c9"
@@
       (reference "IC3") (unit 1) (value "CD4510BE") (footprint "SamacSys_Parts:DIP794W53P254L1930H508Q16N")
     )
-    (path "/d94c84b2-23e1-4bd8-bf01-3a2bfdd61d61"
+    (path "/6f566def-ccf5-4f24-8c95-5a152fda8ef8"
       (reference "J1") (unit 1) (value "CLOCK_IN") (footprint "Connector_Audio:Jack_3.5mm_QingPu_WQP-PJ398SM_Vertical_CircularHoles")
     )
@@
     )
     (path "/b7a58442-8471-47d1-8f65-f9b0cc04ffba"
-      (reference "R5") (unit 1) (value "47K") (footprint "Resistor_THT:R_Axial_DIN0207_L6.3mm_D2.5mm_P7.62mm_Horizontal")
+      (reference "R5") (unit 1) (value "47K") (footprint "Resistor_THT:R_Axial_DIN0204_L3.6mm_D1.6mm_P5.08mm_Horizontal")
     )
     (path "/9e8b7aeb-26a1-4263-8be6-38e156bee711"
@@
     )
     (path "/42763455-1a81-4d1e-bbb6-bc0b264c8fe6"
-      (reference "R7") (unit 1) (value "1K") (footprint "Diode_THT:D_A-405_P7.62mm_Horizontal")
+      (reference "R7") (unit 1) (value "1K") (footprint "Resistor_THT:R_Axial_DIN0204_L3.6mm_D1.6mm_P5.08mm_Horizontal")
     )
     (path "/87febd88-18ef-482e-82ab-3d6176300001"
-      (reference "R8") (unit 1) (value "10k") (footprint "Resistor_SMD:R_0805_2012Metric")
+      (reference "R8") (unit 1) (value "10k") (footprint "Resistor_THT:R_Axial_DIN0204_L3.6mm_D1.6mm_P5.08mm_Horizontal")
     )
     (path "/80f0deea-1d47-466c-b1a1-5c5a371dbe4c"

Commit message: Fix Transitor Logic Add LED Button Datasheet
Connections:
- net GND: now also IC3.15 (CLOCK), Q2.2 (B), SW1.4 (A)
- net at Q2.3 (C), R7.2: no longer SW1.4 (A)
- net CLOCK_IN: no longer names the net of Q1.3 (C), R8.2
- net CLOCK_IN: no longer IC3.15 (CLOCK), Q2.2 (B)
Other:
- note added: "This is backwards, button won't blink, needs to move to emmitter"
- moved on the sheet: Q2, R7
Changed lines of the file:
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@@
   (junction (at 64.77 38.1) (diameter 0) (color 0 0 0 0)
   )
-  (junction (at 190.5 133.35) (diameter 0) (color 0 0 0 0)
-  )
-  (junction (at 246.38 139.7) (diameter 0) (color 0 0 0 0)
-  )
   (junction (at 50.8 176.53) (diameter 0) (color 0 0 0 0)
   )
@@
   (junction (at 226.06 78.74) (diameter 0) (color 0 0 0 0)
   )
+  (junction (at 190.5 148.59) (diameter 0) (color 0 0 0 0)
+  )
   (junction (at 45.72 176.53) (diameter 0) (color 0 0 0 0)
   )
@@
   )
   (junction (at 201.93 76.2) (diameter 0) (color 0 0 0 0)
+  )
+  (junction (at 259.08 142.24) (diameter 0) (color 0 0 0 0)
   )
   (junction (at 226.06 38.1) (diameter 0) (color 0 0 0 0)
@@
     (stroke (width 0) (type default) (color 0 0 0 0))
   )
-  (wire (pts (xy 190.5 146.05) (xy 190.5 149.86))
+  (wire (pts (xy 190.5 146.05) (xy 190.5 148.59))
     (stroke (width 0) (type default) (color 0 0 0 0))
   )
@@
     (stroke (width 0) (type default) (color 0 0 0 0))
   )
-  (wire (pts (xy 190.5 133.35) (xy 190.5 132.08))
+  (wire (pts (xy 190.5 132.08) (xy 190.5 135.89))
     (stroke (width 0) (type default) (color 0 0 0 0))
   )
@@
     (stroke (width 0) (type default) (color 0 0 0 0))
   )
-  (wire (pts (xy 196.85 133.35) (xy 190.5 133.35))
-    (stroke (width 0) (type default) (color 0 0 0 0))
-  )
   (wire (pts (xy 60.96 26.67) (xy 58.42 26.67))
     (stroke (width 0) (type default) (color 0 0 0 0))
@@
     (stroke (width 0) (type default) (color 0 0 0 0))
   )
-  (wire (pts (xy 246.38 129.54) (xy 246.38 139.7))
+  (wire (pts (xy 190.5 148.59) (xy 190.5 149.86))
     (stroke (width 0) (type default) (color 0 0 0 0))
   )
@@
     (stroke (width 0) (type default) (color 0 0 0 0))
   )
-  (wire (pts (xy 236.22 139.7) (xy 237.49 139.7))
+  (wire (pts (xy 259.08 142.24) (xy 266.7 142.24))
+    (stroke (width 0) (type default) (color 0 0 0 0))
+  )
+  (wire (pts (xy 231.14 142.24) (xy 232.41 142.24))
     (stroke (width 0) (type default) (color 0 0 0 0))
   )
@@
     (stroke (width 0) (type default) (color 0 0 0 0))
   )
+  (wire (pts (xy 259.08 129.54) (xy 259.08 142.24))
+    (stroke (width 0) (type default) (color 0 0 0 0))
+  )
   (wire (pts (xy 226.06 38.1) (xy 227.33 38.1))
     (stroke (width 0) (type default) (color 0 0 0 0))
@@
     (stroke (width 0) (type default) (color 0 0 0 0))
   )
+  (wire (pts (xy 198.12 148.59) (xy 190.5 148.59))
+    (stroke (width 0) (type default) (color 0 0 0 0))
+  )
   (wire (pts (xy 198.12 20.32) (xy 198.12 22.86))
     (stroke (width 0) (type default) (color 0 0 0 0))
@@
     (stroke (width 0) (type default) (color 0 0 0 0))
   )
+  (wire (pts (xy 245.11 129.54) (xy 259.08 129.54))
+    (stroke (width 0) (type default) (color 0 0 0 0))
+  )
   (wire (pts (xy 71.12 106.68) (xy 74.93 106.68))
     (stroke (width 0) (type default) (color 0 0 0 0))
@@
     (stroke (width 0) (type default) (color 0 0 0 0))
   )
-  (wire (pts (xy 246.38 129.54) (xy 245.11 129.54))
-    (stroke (width 0) (type default) (color 0 0 0 0))
-  )
   (wire (pts (xy 45.72 176.53) (xy 39.37 176.53))
     (stroke (width 0) (type default) (color 0 0 0 0))
   )
-  (wire (pts (xy 245.11 139.7) (xy 246.38 139.7))
-    (stroke (width 0) (type default) (color 0 0 0 0))
-  )
   (wire (pts (xy 114.3 27.94) (xy 114.3 33.02))
     (stroke (width 0) (type default) (color 0 0 0 0))
@@
     (stroke (width 0) (type default) (color 0 0 0 0))
   )
-  (wire (pts (xy 246.38 139.7) (xy 248.92 139.7))
+  (wire (pts (xy 240.03 142.24) (xy 243.84 142.24))
     (stroke (width 0) (type default) (color 0 0 0 0))
   )
@@
     (stroke (width 0) (type default) (color 0 0 0 0))
   )
-  (wire (pts (xy 190.5 135.89) (xy 190.5 133.35))
-    (stroke (width 0) (type default) (color 0 0 0 0))
-  )
   (wire (pts (xy 115.57 43.18) (xy 110.49 43.18))
     (stroke (width 0) (type default) (color 0 0 0 0))
@@
     (stroke (width 0) (type default) (color 0 0 0 0))
   )
-  (wire (pts (xy 259.08 139.7) (xy 262.89 139.7))
+  (wire (pts (xy 254 142.24) (xy 259.08 142.24))
     (stroke (width 0) (type default) (color 0 0 0 0))
   )
@@
   (text "16 Bars Reset\n" (at 55.88 80.01 0)
     (effects (font (size 2 2)) (justify left bottom))
+  )
+  (text "This is backwards, button won't blink, needs to move to emmitter\n"
+    (at 212.09 110.49 0)
+    (effects (font (size 1.27 1.27)) (justify left bottom))
   )
   (text "Beat Counter" (at 80.01 17.78 0)
@@
     )
   )
-  (global_label "CLOCK_IN" (shape input) (at 196.85 133.35 0) (fields_autoplaced)
+  (global_label "CLOCK_IN" (shape input) (at 198.12 148.59 0) (fields_autoplaced)
     (effects (font (size 1.27 1.27)) (justify left))
-    (property "Intersheet References" "${INTERSHEET_REFS}" (id 0) (at 208.3345 133.2706 0)
+    (property "Intersheet References" "${INTERSHEET_REFS}" (id 0) (at 209.6045 148.5106 0)
       (effects (font (size 1.27 1.27)) (justify left) hide)
     )
@@
     )
   )
-  (global_label "CLOCK_IN" (shape input) (at 254 147.32 270) (fields_autoplaced)
+  (global_label "CLOCK_IN" (shape input) (at 248.92 149.86 270) (fields_autoplaced)
     (effects (font (size 1.27 1.27)) (justify right))
-    (property "Intersheet References" "${INTERSHEET_REFS}" (id 0) (at 254.0794 158.8045 90)
+    (property "Intersheet References" "${INTERSHEET_REFS}" (id 0) (at 248.9994 161.3445 90)
       (effects (font (size 1.27 1.27)) (justify right) hide)
     )
@@
     (pin "3")
   )
-  (symbol (lib_id "Transistor_BJT:2N3904") (at 254 142.24 90) (unit 1)
-    (in_bom yes) (on_board yes) (fields_autoplaced)
-    (property "Reference" "Q2" (id 0) (at 252.7299 137.16 0)
+  (symbol (lib_id "Transistor_BJT:2N3904") (at 248.92 144.78 90) (unit 1)
+    (in_bom yes) (on_board yes)
+    (property "Reference" "Q2" (id 0) (at 255.27 139.7 90)
       (effects (font (size 1.27 1.27)) (justify left))
     )
-    (property "Value" "2N3904" (id 1) (at 255.2699 137.16 0)
+    (property "Value" "2N3904" (id 1) (at 255.27 137.16 90)
       (effects (font (size 1.27 1.27)) (justify left))
     )
-    (property "Footprint" "Package_TO_SOT_THT:TO-92_Inline" (id 2) (at 255.905 137.16 0)
+    (property "Footprint" "Package_TO_SOT_THT:TO-92_Inline" (id 2) (at 250.825 139.7 0)
       (effects (font (size 1.27 1.27) italic) (justify left) hide)
     )
-    (property "Datasheet" "https://www.onsemi.com/pub/Collateral/2N3903-D.PDF" (id 3) (at 254 142.24 0)
+    (property "Datasheet" "https://www.onsemi.com/pub/Collateral/2N3903-D.PDF" (id 3) (at 248.92 144.78 0)
       (effects (font (size 1.27 1.27)) (justify left) hide)
     )
@@
     (pin "2")
   )
-  (symbol (lib_id "Device:R") (at 241.3 139.7 90) (unit 1)
-    (in_bom yes) (on_board yes) (fields_autoplaced)
-    (property "Reference" "R7" (id 0) (at 242.5701 142.24 0)
+  (symbol (lib_id "Device:R") (at 236.22 142.24 90) (unit 1)
+    (in_bom yes) (on_board yes)
+    (property "Reference" "R7" (id 0) (at 234.95 144.7799 90)
       (effects (font (size 1.27 1.27)) (justify right))
     )
-    (property "Value" "1K" (id 1) (at 240.0301 142.24 0)
+    (property "Value" "1K" (id 1) (at 234.95 147.3199 90)
       (effects (font (size 1.27 1.27)) (justify right))
     )
-    (property "Footprint" "Resistor_THT:R_Axial_DIN0204_L3.6mm_D1.6mm_P5.08mm_Horizontal" (id 2) (at 241.3 141.478 90)
-      (effects (font (size 1.27 1.27)) hide)
-    )
-    (property "Datasheet" "~" (id 3) (at 241.3 139.7 0)
+    (property "Footprint" "Resistor_THT:R_Axial_DIN0204_L3.6mm_D1.6mm_P5.08mm_Horizontal" (id 2) (at 236.22 144.018 90)
+      (effects (font (size 1.27 1.27)) hide)
+    )
+    (property "Datasheet" "~" (id 3) (at 236.22 142.24 0)
       (effects (font (size 1.27 1.27)) hide)
     )
@@
     (pin "2")
   )
-  (symbol (lib_id "power:+12V") (at 236.22 139.7 90) (unit 1)
-    (in_bom yes) (on_board yes) (fields_autoplaced)
-    (property "Reference" "#PWR016" (id 0) (at 240.03 139.7 0)
-      (effects (font (size 1.27 1.27)) hide)
-    )
-    (property "Value" "+12V" (id 1) (at 231.14 139.7 0))
-    (property "Footprint" "" (id 2) (at 236.22 139.7 0)
-      (effects (font (size 1.27 1.27)) hide)
-    )
-    (property "Datasheet" "" (id 3) (at 236.22 139.7 0)
+  (symbol (lib_id "power:+12V") (at 231.14 142.24 90) (unit 1)
+    (in_bom yes) (on_board yes)
+    (property "Reference" "#PWR016" (id 0) (at 234.95 142.24 0)
+      (effects (font (size 1.27 1.27)) hide)
+    )
+    (property "Value" "+12V" (id 1) (at 226.06 142.24 90))
+    (property "Footprint" "" (id 2) (at 231.14 142.24 0)
+      (effects (font (size 1.27 1.27)) hide)
+    )
+    (property "Datasheet" "" (id 3) (at 231.14 142.24 0)
       (effects (font (size 1.27 1.27)) hide)
     )
@@
     (pin "1")
   )
-  (symbol (lib_id "power:GND") (at 262.89 139.7 90) (unit 1)
-    (in_bom yes) (on_board yes) (fields_autoplaced)
-    (property "Reference" "#PWR019" (id 0) (at 269.24 139.7 0)
-      (effects (font (size 1.27 1.27)) hide)
-    )
-    (property "Value" "GND" (id 1) (at 267.97 139.7 0))
-    (property "Footprint" "" (id 2) (at 262.89 139.7 0)
-      (effects (font (size 1.27 1.27)) hide)
-    )
-    (property "Datasheet" "" (id 3) (at 262.89 139.7 0)
-      (effects (font (size 1.27 1.27)) hide)
-    )
+  (symbol (lib_id "power:GND") (at 266.7 142.24 90) (unit 1)
+    (in_bom yes) (on_board yes) (fields_autoplaced)
+    (property "Reference" "#PWR019" (id 0) (at 273.05 142.24 0)
+      (effects (font (size 1.27 1.27)) hide)
+    )
+    (property "Value" "GND" (id 1) (at 271.78 142.24 0))
+    (property "Footprint" "" (id 2) (at 266.7 142.24 0)
+      (effects (font (size 1.27 1.27)) hide)
+    )
+    (property "Datasheet" "" (id 3) (at 266.7 142.24 0)
+      (effects (font (size 1.27 1.27)) hide)
+    )

Commit message: Surface Mount Resistors and Caps, fix 7segment footprint
Parts:
- R10, R11, R13, R14: value R -> 10K
- R12, R15: value R -> 4.7K
Changed lines of the file:
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@@
     (in_bom yes) (on_board yes) (fields_autoplaced)
     (property "Reference" "R14" (id 0) (at 78.74 100.33 90))
-    (property "Value" "R" (id 1) (at 78.74 102.87 90))
+    (property "Value" "10K" (id 1) (at 78.74 102.87 90))
     (property "Footprint" "Resistor_THT:R_Axial_DIN0204_L3.6mm_D1.6mm_P5.08mm_Horizontal" (id 2) (at 78.74 108.458 90)
       (effects (font (size 1.27 1.27)) hide)
@@
     (in_bom yes) (on_board yes) (fields_autoplaced)
     (property "Reference" "R10" (id 0) (at 41.91 86.36 90))
-    (property "Value" "R" (id 1) (at 41.91 88.9 90))
+    (property "Value" "10K" (id 1) (at 41.91 88.9 90))
     (property "Footprint" "Resistor_THT:R_Axial_DIN0204_L3.6mm_D1.6mm_P5.08mm_Horizontal" (id 2) (at 41.91 94.488 90)
       (effects (font (size 1.27 1.27)) hide)
@@
     (in_bom yes) (on_board yes) (fields_autoplaced)
     (property "Reference" "R11" (id 0) (at 41.91 99.06 90))
-    (property "Value" "R" (id 1) (at 41.91 101.6 90))
+    (property "Value" "10K" (id 1) (at 41.91 101.6 90))
     (property "Footprint" "Resistor_THT:R_Axial_DIN0204_L3.6mm_D1.6mm_P5.08mm_Horizontal" (id 2) (at 41.91 107.188 90)
       (effects (font (size 1.27 1.27)) hide)
@@
       (effects (font (size 1.27 1.27)) (justify left))
     )
-    (property "Value" "R" (id 1) (at 55.88 119.3799 0)
+    (property "Value" "4.7K" (id 1) (at 55.88 119.3799 0)
       (effects (font (size 1.27 1.27)) (justify left))
     )
@@
       (effects (font (size 1.27 1.27)) (justify left))
     )
-    (property "Value" "R" (id 1) (at 92.71 120.6499 0)
+    (property "Value" "4.7K" (id 1) (at 92.71 120.6499 0)
       (effects (font (size 1.27 1.27)) (justify left))
     )
@@
     (in_bom yes) (on_board yes) (fields_autoplaced)
     (property "Reference" "R13" (id 0) (at 78.74 87.63 90))
-    (property "Value" "R" (id 1) (at 78.74 90.17 90))
+    (property "Value" "10K" (id 1) (at 78.74 90.17 90))
     (property "Footprint" "Resistor_THT:R_Axial_DIN0204_L3.6mm_D1.6mm_P5.08mm_Horizontal" (id 2) (at 78.74 95.758 90)
       (effects (font (size 1.27 1.27)) hide)
@@
     )
     (path "/3806a02f-aee2-4d3b-926e-623af1f9ae30"
-      (reference "R10") (unit 1) (value "R") (footprint "Resistor_THT:R_Axial_DIN0204_L3.6mm_D1.6mm_P5.08mm_Horizontal")
+      (reference "R10") (unit 1) (value "10K") (footprint "Resistor_THT:R_Axial_DIN0204_L3.6mm_D1.6mm_P5.08mm_Horizontal")
     )
     (path "/5715c485-4223-439b-99db-4c09f36dc03d"
-      (reference "R11") (unit 1) (value "R") (footprint "Resistor_THT:R_Axial_DIN0204_L3.6mm_D1.6mm_P5.08mm_Horizontal")
+      (reference "R11") (unit 1) (value "10K") (footprint "Resistor_THT:R_Axial_DIN0204_L3.6mm_D1.6mm_P5.08mm_Horizontal")
     )
     (path "/6c329504-5ebc-4d7c-9138-4b45f007bfb0"
-      (reference "R12") (unit 1) (value "R") (footprint "Resistor_THT:R_Axial_DIN0204_L3.6mm_D1.6mm_P5.08mm_Horizontal")
+      (reference "R12") (unit 1) (value "4.7K") (footprint "Resistor_THT:R_Axial_DIN0204_L3.6mm_D1.6mm_P5.08mm_Horizontal")
     )
     (path "/a3aca66e-0260-49f9-949e-e0960bc113f0"
-      (reference "R13") (unit 1) (value "R") (footprint "Resistor_THT:R_Axial_DIN0204_L3.6mm_D1.6mm_P5.08mm_Horizontal")
+      (reference "R13") (unit 1) (value "10K") (footprint "Resistor_THT:R_Axial_DIN0204_L3.6mm_D1.6mm_P5.08mm_Horizontal")
     )
     (path "/2204773c-5355-4949-8953-4afa6b7c31c8"
-      (reference "R14") (unit 1) (value "R") (footprint "Resistor_THT:R_Axial_DIN0204_L3.6mm_D1.6mm_P5.08mm_Horizontal")
+      (reference "R14") (unit 1) (value "10K") (footprint "Resistor_THT:R_Axial_DIN0204_L3.6mm_D1.6mm_P5.08mm_Horizontal")
     )
     (path "/918017a1-9a8a-4832-8382-dad331e88e6c"
-      (reference "R15") (unit 1) (value "R") (footprint "Resistor_THT:R_Axial_DIN0204_L3.6mm_D1.6mm_P5.08mm_Horizontal")
+      (reference "R15") (unit 1) (value "4.7K") (footprint "Resistor_THT:R_Axial_DIN0204_L3.6mm_D1.6mm_P5.08mm_Horizontal")
     )
     (path "/cb2a04d5-6f2d-4dd0-95e6-7d34ea886b6a"
