File: 16Bars.kicad_pcb (KiCad board)
At the start: 2 copper layers, 28.5 x 105 mm, 49 parts, among them IC1 CD4033BE, IC2 CD4033BE, IC3 CD4510BE, IC4 CD4510BE, IC5 CD4510BE, J1 3.5mm_Mono_Switched, J2 Conn_02x05_Odd_Even, Q1 2N3904, Q2 2N3904, Q3 2N3904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

Commit message: Finish PCB Layout
Parts:
- removed G***: LOGO, ArtworkFootprints:SixteenWinds
- moved Q1 52.3 mm to (59.8, 61.2)
- moved R19 51.6 mm to (63.8, 63.0), turned to 180 degrees
- moved R17 51.5 mm to (63.5, 59.8)
- moved R16 42.4 mm to (63.5, 58.2)
- moved C11 32.2 mm to (72.5, 49.5)
- moved D1 31.8 mm to (68.5, 49.2)
- moved R5 29.6 mm to (64.2, 49.5), turned to 180 degrees
- moved Q2 20.0 mm to (81.6, 60.5)
- moved R11 16.0 mm to (77.0, 63.2), turned to 180 degrees
- moved R14 13.6 mm to (77.0, 62.0), turned to 180 degrees
- moved R20 13.4 mm to (71.5, 59.8)
- moved R9 12.8 mm to (75.0, 90.5)
- moved Q3 12.0 mm to (67.2, 61.2), turned to 180 degrees
- moved R8 9.12 mm to (64.0, 88.0)
- moved R7 8.25 mm to (64.0, 90.5)
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Routing:
- net +12V: track 6.63 -> 193.8 mm, vias 0 -> 1
- net /RESET: track 5.04 -> 99.1 mm, vias 0 -> 1
- net CLOCK_IN: track 0.00 -> 88.8 mm
- net CLOCK_BAR: track 0.00 -> 76.2 mm, vias 0 -> 1
- net /8Beats/Bar: track 0.00 -> 72.9 mm
- net /4Beats/Bar: track 0.00 -> 51.8 mm
- net /16Bars: track 0.00 -> 33.0 mm
- net GND: track 0.00 -> 28.6 mm, vias 0 -> 2
- net Net-(Q2-Pad2): track 0.00 -> 27.6 mm
- net /8Bars: track 0.00 -> 25.4 mm
- net CARRY_1: track 0.00 -> 21.5 mm
- net Net-(C11-Pad1): track 0.00 -> 17.7 mm
- net /BarCountCarry: track 0.00 -> 14.3 mm
- net Net-(Q1-Pad2): track 0.00 -> 6.07 mm
- net Net-(R15-Pad2): track 0.00 -> 5.34 mm
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- added copper zone on F.Cu, net GND

Commit message: Fix DRC errors
Routing:
- net /RESET: track 99.1 -> 101.6 mm, vias 1 -> 2
- net GND: track 28.6 -> 29.9 mm
- net Net-(Q2-Pad2): track 27.6 -> 28.1 mm
