File: LEDShieldPractice/Panel/LedPracticePanel/LedPracticePanel.kicad_pcb (KiCad board)
At the start: 2 copper layers, 40.3 x 39.7 mm, 7 parts

Commit message: OshPark AfterDark Sheep Panel
Parts:
- removed the G*** at (32.1, 31.3)
- removed the G*** at (31.4, 31.3)
- added G***: LOGO, ArtworkFootprints:SheepCopper, F.Cu at (33.0, 30.5)
- moved G*** 0.50 mm to (31.9, 31.3)
Routing:
- removed copper zone on F.Cu, net (none)
- removed copper zone on F.Cu, net GND
Other:
- board text removed: "ubersheep"
