File: LEDShieldPractice/LEDShieldPractice.kicad_sch (KiCad schematic)
At the start: 11 parts, among them J1 Conn_02x05_Odd_Even, J2 CLOCK_IN, Q1 2N3904

Commit message: Resize ClockBlink PCB
Connections:
- net -12V: no longer names the net of J1.10 (Pin_10)
- net -12V: no longer J1.9 (Pin_9)
- no-connect marks 2 -> 3
Other:
- note added: "-12V"
Changed lines of the file:
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@@
   (junction (at 132.08 106.68) (diameter 0) (color 0 0 0 0)
   )
-  (junction (at 144.78 111.76) (diameter 0) (color 0 0 0 0)
-  )
   (junction (at 158.75 106.68) (diameter 0) (color 0 0 0 0)
   )
@@
   (junction (at 144.78 106.68) (diameter 0) (color 0 0 0 0)
   )
-  (no_connect (at 151.13 111.76))
+  (no_connect (at 144.78 111.76))
+  (no_connect (at 132.08 111.76))
   (no_connect (at 109.22 48.26))
-  (wire (pts (xy 132.08 113.03) (xy 132.08 111.76))
-    (stroke (width 0) (type default) (color 0 0 0 0))
-  )
   (wire (pts (xy 132.08 109.22) (xy 132.08 106.68))
     (stroke (width 0) (type default) (color 0 0 0 0))
@@
     (stroke (width 0) (type default) (color 0 0 0 0))
   )
-  (wire (pts (xy 144.78 111.76) (xy 151.13 111.76))
-    (stroke (width 0) (type default) (color 0 0 0 0))
-  )
   (wire (pts (xy 151.13 101.6) (xy 158.75 101.6))
     (stroke (width 0) (type default) (color 0 0 0 0))
@@
   )
   (wire (pts (xy 200.66 144.78) (xy 200.66 147.32))
-    (stroke (width 0) (type default) (color 0 0 0 0))
-  )
-  (wire (pts (xy 144.78 113.03) (xy 132.08 113.03))
-    (stroke (width 0) (type default) (color 0 0 0 0))
-  )
-  (wire (pts (xy 144.78 111.76) (xy 144.78 113.03))
     (stroke (width 0) (type default) (color 0 0 0 0))
   )
@@
     (effects (font (size 1.524 1.524) (thickness 0.3048) bold) (justify right bottom))
   )
+  (text "-12V" (at 135.89 116.84 0)
+    (effects (font (size 1.27 1.27)) (justify left bottom))
+  )
   (label "+12V" (at 162.56 101.6 0)
-    (effects (font (size 1.27 1.27)) (justify left bottom))
-  )
-  (label "-12V" (at 151.13 111.76 0)
     (effects (font (size 1.27 1.27)) (justify left bottom))
   )
@@
   (symbol (lib_id "power:GND") (at 173.99 116.84 0) (unit 1)
     (in_bom yes) (on_board yes) (fields_autoplaced)
-    (property "Reference" "#PWR?" (id 0) (at 173.99 123.19 0)
+    (property "Reference" "#PWR0101" (id 0) (at 173.99 123.19 0)
       (effects (font (size 1.27 1.27)) hide)
     )
@@
   (symbol (lib_id "power:GND") (at 215.9 116.84 0) (unit 1)
     (in_bom yes) (on_board yes) (fields_autoplaced)
-    (property "Reference" "#PWR?" (id 0) (at 215.9 123.19 0)
+    (property "Reference" "#PWR0102" (id 0) (at 215.9 123.19 0)
       (effects (font (size 1.27 1.27)) hide)
     )
@@
     )
     (path "/12e7e1e5-156c-4508-bb16-ff0d257426f0"
-      (reference "#PWR?") (unit 1) (value "GND") (footprint "")
+      (reference "#PWR0101") (unit 1) (value "GND") (footprint "")
     )
     (path "/1a6ed829-b2ec-4ab8-821d-044212b78fcd"
-      (reference "#PWR?") (unit 1) (value "GND") (footprint "")
+      (reference "#PWR0102") (unit 1) (value "GND") (footprint "")
     )
     (path "/b72fc618-8796-405b-bf22-185e95a533a3"

Commit message: Update LED Shield Practice
Updated footprints for flush fitting resistors and reran traces. Build 2nd board from last years run, changed led resistors from 500 to 2k, 500 burned out leds with 12v.
Board works but the clock led is lit and turns off when it receives a signal, the transistor is acting as a logic NOT, unsure how to debug, need time on the breadboard.
Parts:
- R1, R2: value 500 -> 2000; footprint Resistor_THT:R_Axial_DIN0204_L3.6mm_D1.6mm_P5.08mm_Horizontal -> Resistor_THT:R_Axial_DIN0207_L6.3mm_D2.5mm_P10.16mm_Horizontal
- R3, R4: footprint Resistor_THT:R_Axial_DIN0204_L3.6mm_D1.6mm_P5.08mm_Horizontal -> Resistor_THT:R_Axial_DIN0207_L6.3mm_D2.5mm_P10.16mm_Horizontal
Changed lines of the file:
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@@
       (effects (font (size 1.27 1.27)) (justify left))
     )
-    (property "Value" "500" (id 1) (at 176.53 110.4899 0)
-      (effects (font (size 1.27 1.27)) (justify left))
-    )
-    (property "Footprint" "Resistor_THT:R_Axial_DIN0204_L3.6mm_D1.6mm_P5.08mm_Horizontal" (id 2) (at 172.212 109.22 90)
+    (property "Value" "2000" (id 1) (at 176.53 110.4899 0)
+      (effects (font (size 1.27 1.27)) (justify left))
+    )
+    (property "Footprint" "Resistor_THT:R_Axial_DIN0207_L6.3mm_D2.5mm_P10.16mm_Horizontal" (id 2) (at 172.212 109.22 90)
       (effects (font (size 1.27 1.27)) hide)
     )
@@
   )
   (symbol (lib_id "Device:LED") (at 215.9 96.52 90) (unit 1)
-    (in_bom yes) (on_board yes) (fields_autoplaced)
+    (in_bom yes) (on_board yes)
     (property "Reference" "D2" (id 0) (at 219.71 96.8374 90)
       (effects (font (size 1.27 1.27)) (justify right))
@@
       (effects (font (size 1.27 1.27)) (justify left))
     )
-    (property "Footprint" "Resistor_THT:R_Axial_DIN0204_L3.6mm_D1.6mm_P5.08mm_Horizontal" (id 2) (at 235.712 129.54 90)
+    (property "Footprint" "Resistor_THT:R_Axial_DIN0207_L6.3mm_D2.5mm_P10.16mm_Horizontal" (id 2) (at 235.712 129.54 90)
       (effects (font (size 1.27 1.27)) hide)
     )
@@
     (property "Reference" "R3" (id 0) (at 222.25 139.7 90))
     (property "Value" "47K" (id 1) (at 222.25 142.24 90))
-    (property "Footprint" "Resistor_THT:R_Axial_DIN0204_L3.6mm_D1.6mm_P5.08mm_Horizontal" (id 2) (at 222.25 140.462 90)
+    (property "Footprint" "Resistor_THT:R_Axial_DIN0207_L6.3mm_D2.5mm_P10.16mm_Horizontal" (id 2) (at 222.25 140.462 90)
       (effects (font (size 1.27 1.27)) hide)
     )
@@
   )
   (symbol (lib_id "Device:R") (at 215.9 109.22 0) (unit 1)
-    (in_bom yes) (on_board yes) (fields_autoplaced)
+    (in_bom yes) (on_board yes)
     (property "Reference" "R2" (id 0) (at 218.44 107.9499 0)
       (effects (font (size 1.27 1.27)) (justify left))
     )
-    (property "Value" "500" (id 1) (at 218.44 110.4899 0)
-      (effects (font (size 1.27 1.27)) (justify left))
-    )
-    (property "Footprint" "Resistor_THT:R_Axial_DIN0204_L3.6mm_D1.6mm_P5.08mm_Horizontal" (id 2) (at 214.122 109.22 90)
+    (property "Value" "2000" (id 1) (at 218.44 110.4899 0)
+      (effects (font (size 1.27 1.27)) (justify left))
+    )
+    (property "Footprint" "Resistor_THT:R_Axial_DIN0207_L6.3mm_D2.5mm_P10.16mm_Horizontal" (id 2) (at 214.122 109.22 90)
       (effects (font (size 1.27 1.27)) hide)
     )
@@
     )
     (path "/188aa0aa-34a1-4369-a101-253e9bd6c5f8"
-      (reference "R1") (unit 1) (value "500") (footprint "Resistor_THT:R_Axial_DIN0204_L3.6mm_D1.6mm_P5.08mm_Horizontal")
+      (reference "R1") (unit 1) (value "2000") (footprint "Resistor_THT:R_Axial_DIN0207_L6.3mm_D2.5mm_P10.16mm_Horizontal")
     )
     (path "/f5f27541-ea3f-424f-97c0-1482a2b990db"
-      (reference "R2") (unit 1) (value "500") (footprint "Resistor_THT:R_Axial_DIN0204_L3.6mm_D1.6mm_P5.08mm_Horizontal")
+      (reference "R2") (unit 1) (value "2000") (footprint "Resistor_THT:R_Axial_DIN0207_L6.3mm_D2.5mm_P10.16mm_Horizontal")
     )
     (path "/becc5a78-13b1-4e67-8592-989db2beb20d"
-      (reference "R3") (unit 1) (value "47K") (footprint "Resistor_THT:R_Axial_DIN0204_L3.6mm_D1.6mm_P5.08mm_Horizontal")
+      (reference "R3") (unit 1) (value "47K") (footprint "Resistor_THT:R_Axial_DIN0207_L6.3mm_D2.5mm_P10.16mm_Horizontal")
     )
     (path "/999ec242-2b7a-44b5-b5e9-e2fb89a4fff8"
-      (reference "R4") (unit 1) (value "10k") (footprint "Resistor_THT:R_Axial_DIN0204_L3.6mm_D1.6mm_P5.08mm_Horizontal")
-    )
-  )
+      (reference "R4") (unit 1) (value "10k") (footprint "Resistor_THT:R_Axial_DIN0207_L6.3mm_D2.5mm_P10.16mm_Horizontal")
+    )
+  )

Commit message: Update LED Panel layout, added panel with mouse bites.
Connections:
- net +12V: now also Q1.3 (C); no longer R4.1
- net CLOCK: now also Q1.1 (E), R2.1, R4.1; no longer D2.2 (A), Q1.3 (C), R4.2
- net GND: now also D2.1 (K), R4.2; no longer Q1.1 (E), R2.2
- net -12V: now reaches J1.10 (Pin_10)
- net -12V: now also J1.9 (Pin_9)
- new net: D2.2 (A), R2.2
- no-connect marks 3 -> 1

Commit message: Fix transistor logic. TODO resistor values.
Other:
- note removed: "-12V"
Changed lines of the file:
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@@
     (effects (font (size 1.524 1.524) (thickness 0.3048) bold) (justify right bottom))
-  )
-  (text "-12V" (at 135.89 116.84 0)
-    (effects (font (size 1.27 1.27)) (justify left bottom))
   )
   (label "+12V" (at 162.56 101.6 0)
@@
       (reference "#PWR05") (unit 1) (value "+12V") (footprint "")
     )
-    (path "/2f312f60-80b4-4a8a-b378-5a3d48c8a106"
-      (reference "#PWR06") (unit 1) (value "GND") (footprint "")
-    )
     (path "/12e7e1e5-156c-4508-bb16-ff0d257426f0"
