File: Miduino/Miduino.kicad_sch (KiCad schematic)
At the start: 9 parts

Commit message: Miduino TODOs
Parts:
- gave numbers to parts that had none: 8
Other:
- note added: "TODO assign footprints"
- note removed: "TODO how to switch off Midi for USB programming on RX?"
Changed lines of the file:
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@@
     (stroke (width 0) (type default) (color 0 0 0 0))
   )
-  (text "TODO how to switch off Midi for USB programming on RX?"
-    (at 127 118.11 0)
+  (text "TODO assign footprints\n" (at 55.88 116.84 0)
     (effects (font (size 1.27 1.27)) (justify left bottom))
   )
@@
   (symbol (lib_id "4ms_Resistor:470R_0603") (at 120.65 99.06 0) (unit 1)
     (in_bom yes) (on_board yes) (fields_autoplaced)
-    (property "Reference" "R?" (id 0) (at 123.19 97.7899 0)
+    (property "Reference" "R3" (id 0) (at 123.19 97.7899 0)
       (effects (font (size 1.27 1.27)) (justify left))
     )
@@
   (symbol (lib_id "Switch:SW_DPDT_x2") (at 50.8 105.41 0) (unit 2)
     (in_bom yes) (on_board yes) (fields_autoplaced)
-    (property "Reference" "SW?" (id 0) (at 50.8 97.79 0))
+    (property "Reference" "SW1" (id 0) (at 50.8 97.79 0))
     (property "Value" "SW_DPDT_x2" (id 1) (at 50.8 100.33 0))
     (property "Footprint" "" (id 2) (at 50.8 105.41 0)
@@
   (symbol (lib_id "4ms_Resistor:1k_0603") (at 113.03 107.95 0) (unit 1)
     (in_bom yes) (on_board yes) (fields_autoplaced)
-    (property "Reference" "R?" (id 0) (at 115.57 106.6799 0)
+    (property "Reference" "R2" (id 0) (at 115.57 106.6799 0)
       (effects (font (size 1.27 1.27)) (justify left))
     )
@@
   (symbol (lib_id "Isolator:6N138") (at 99.06 101.6 0) (unit 1)
     (in_bom yes) (on_board yes) (fields_autoplaced)
-    (property "Reference" "U?" (id 0) (at 99.06 88.9 0))
+    (property "Reference" "U1" (id 0) (at 99.06 88.9 0))
     (property "Value" "6N138" (id 1) (at 99.06 91.44 0))
     (property "Footprint" "" (id 2) (at 106.426 109.22 0)
@@
   (symbol (lib_id "4ms_Power-symbol:GND") (at 106.68 118.11 0) (unit 1)
     (in_bom yes) (on_board yes) (fields_autoplaced)
-    (property "Reference" "#PWR?" (id 0) (at 106.68 124.46 0)
+    (property "Reference" "#PWR0102" (id 0) (at 106.68 124.46 0)
       (effects (font (size 1.27 1.27)) hide)
     )
@@
   (symbol (lib_id "Switch:SW_DPDT_x2") (at 53.34 92.71 0) (unit 1)
     (in_bom yes) (on_board yes) (fields_autoplaced)
-    (property "Reference" "SW?" (id 0) (at 53.34 85.09 0))
+    (property "Reference" "SW1" (id 0) (at 53.34 85.09 0))
     (property "Value" "SW_DPDT_x2" (id 1) (at 53.34 87.63 0))
     (property "Footprint" "" (id 2) (at 53.34 92.71 0)
@@
   (symbol (lib_id "4ms_Power-symbol:+5V") (at 120.65 95.25 0) (unit 1)
     (in_bom yes) (on_board yes) (fields_autoplaced)
-    (property "Reference" "#PWR?" (id 0) (at 120.65 99.06 0)
+    (property "Reference" "#PWR0101" (id 0) (at 120.65 99.06 0)
       (effects (font (size 1.27 1.27)) hide)
     )
@@
   (symbol (lib_id "Switch:SW_SPST") (at 125.73 104.14 0) (unit 1)
     (in_bom yes) (on_board yes) (fields_autoplaced)
-    (property "Reference" "SW?" (id 0) (at 125.73 97.79 0))
+    (property "Reference" "SW2" (id 0) (at 125.73 97.79 0))
     (property "Value" "SW_SPST" (id 1) (at 125.73 100.33 0))
     (property "Footprint" "" (id 2) (at 125.73 104.14 0)
@@
   (symbol (lib_id "4ms_Resistor:220R_0603") (at 80.01 96.52 90) (unit 1)
     (in_bom yes) (on_board yes) (fields_autoplaced)
-    (property "Reference" "R?" (id 0) (at 80.01 90.17 90))
+    (property "Reference" "R1" (id 0) (at 80.01 90.17 90))
     (property "Value" "220R_0603" (id 1) (at 80.01 99.06 90)
       (effects (font (size 1.27 1.27)) hide)
@@
   (symbol (lib_id "4ms_Jack:3.5mm_Stereo") (at 38.1 100.33 0) (unit 1)
     (in_bom yes) (on_board yes) (fields_autoplaced)
-    (property "Reference" "J?" (id 0) (at 38.735 90.17 0)
+    (property "Reference" "J1" (id 0) (at 38.735 90.17 0)
       (effects (font (size 1.524 1.524)))
     )
@@
   (symbol (lib_id "4ms_Diode:1N914BWS") (at 83.82 100.33 270) (unit 1)
     (in_bom yes) (on_board yes)
-    (property "Reference" "D?" (id 0) (at 82.55 107.95 90)
+    (property "Reference" "D1" (id 0) (at 82.55 107.95 90)
       (effects (font (size 1.27 1.27)) (justify left))
     )
@@
   )
   (symbol_instances
+    (path "/ba9fd67a-72b6-4618-a24e-a295aa8f7562"
+      (reference "#PWR0101") (unit 1) (value "+5V") (footprint "")
+    )
     (path "/a7684d27-7355-46b0-8d10-287b5e8c3422"
-      (reference "#PWR?") (unit 1) (value "GND") (footprint "")
-    )
-    (path "/ba9fd67a-72b6-4618-a24e-a295aa8f7562"
-      (reference "#PWR?") (unit 1) (value "+5V") (footprint "")
+      (reference "#PWR0102") (unit 1) (value "GND") (footprint "")
     )
     (path "/fd4cd5da-c64d-4f44-a60c-dd9716e0e239"
-      (reference "D?") (unit 1) (value "1N914BWS") (footprint "4ms_Diode:D_SOD-323F")
+      (reference "D1") (unit 1) (value "1N914BWS") (footprint "4ms_Diode:D_SOD-323F")
     )
     (path "/eeb87454-981e-4f6e-abec-27786ad762d7"
-      (reference "J?") (unit 1) (value "3.5mm_Stereo") (footprint "4ms_Jack:EighthInch_Stereo_PJ366ST")
+      (reference "J1") (unit 1) (value "3.5mm_Stereo") (footprint "4ms_Jack:EighthInch_Stereo_PJ366ST")
+    )
+    (path "/dcf828fc-8f65-41d7-9aa2-756a8377ae36"
+      (reference "R1") (unit 1) (value "220R_0603") (footprint "4ms_Resistor:R_0603")
+    )
+    (path "/7ba77f6f-f70c-45dc-82b9-70d30eb8bd25"
+      (reference "R2") (unit 1) (value "1k_0603") (footprint "4ms_Resistor:R_0603")
     )
     (path "/04d6273a-6be9-4139-a5eb-793ecc8c0d0e"
-      (reference "R?") (unit 1) (value "470R_0603") (footprint "4ms_Resistor:R_0603")
-    )
-    (path "/7ba77f6f-f70c-45dc-82b9-70d30eb8bd25"
-      (reference "R?") (unit 1) (value "1k_0603") (footprint "4ms_Resistor:R_0603")
-    )
-    (path "/dcf828fc-8f65-41d7-9aa2-756a8377ae36"
-      (reference "R?") (unit 1) (value "220R_0603") (footprint "4ms_Resistor:R_0603")
+      (reference "R3") (unit 1) (value "470R_0603") (footprint "4ms_Resistor:R_0603")
     )
     (path "/aa43ebed-adfc-4dab-b4ce-d6020c1d6141"
-      (reference "SW?") (unit 1) (value "SW_DPDT_x2") (footprint "")
+      (reference "SW1") (unit 1) (value "SW_DPDT_x2") (footprint "")
+    )
+    (path "/60f23abb-e807-43fb-99de-c95a00873103"
+      (reference "SW1") (unit 2) (value "SW_DPDT_x2") (footprint "")
     )
     (path "/d0b0afaf-73f9-4e08-91d2-d4e00a2a1478"
-      (reference "SW?") (unit 1) (value "SW_SPST") (footprint "")
-    )
-    (path "/60f23abb-e807-43fb-99de-c95a00873103"
-      (reference "SW?") (unit 2) (value "SW_DPDT_x2") (footprint "")
+      (reference "SW2") (unit 1) (value "SW_SPST") (footprint "")
     )
     (path "/84e376e1-bc27-4a2e-8002-707d90c8c085"
-      (reference "U?") (unit 1) (value "6N138") (footprint "")
-    )
-  )
+      (reference "U1") (unit 1) (value "6N138") (footprint "")
+    )
+  )
