File: Panel/Panel.kicad_pcb (KiCad board)
At the start: 2 copper layers, 30 x 128.5 mm, 6 parts

Commit message: v3.1
Parts:
- removed the ? at (59.6, 132.2)
- removed the ? at (67.4, 160.0)
- removed the REF** at (69.5, 56.9)
- removed the REF** at (52.4, 37.5)
- removed the REF** at (51.1, 53.4)
- removed the Ref** at (53.6, 160.5)
- added ?: , , F.Cu at (82.8, 97.0)
- added ?: , , F.Cu at (99.1, 162.2)
- added ?: , , F.Cu at (82.8, 83.3)
- added REF**: MountingHole, MountingHole:MountingHole_3.2mm_M3, F.Cu at (82.8, 69.6)
- added REF**: MountingHole_3.2mm_M3, MountingHole:MountingHole_3.2mm_M3, F.Cu at (84.1, 39.7)
- added REF**: MountingHole, MountingHole:MountingHole_3.2mm_M3, F.Cu at (101.1, 59.1)
- added REF**: MountingHole, MountingHole:MountingHole_3.2mm_M3, F.Cu at (82.8, 55.6)
- added Ref**: Val**, LogoFootprints:sedecim-modios-humane-jenson, F.Cu at (98.7, 51.3)
- added Ref**: Val**, LogoFootprints:16WindsLogoJuly2023-12mm-RightSide, F.Cu at (122.1, 164.6)
- added Ref**: Val**, LogoFootprints:aparticas-glyphs-humane-jenson, F.Cu at (92.2, 46.9)
- added Ref**: Val**, LogoFootprints:16WindsLogoJuly2023-12mm, F.Cu at (96.3, 164.6)
Other:
- outline, holes or cut-outs redrawn

Commit message: v3.1 Fabrication for PCB and Panel
Parts:
- removed the Ref** at (98.7, 51.3)
- removed the Ref** at (92.2, 46.9)
- added REF**: 16W-Input, Footprints:16W-Input, F.Cu at (82.8, 55.6)
- added REF**: 16W-Output, Footprints:16W-Output, F.Cu at (82.8, 97.0)
- added REF**: 16W-Output, Footprints:16W-Output, F.Cu at (82.8, 83.3)
- added REF**: 16W-Output, Footprints:16W-Output, F.Cu at (82.8, 69.6)
- added Ref**: Val**, Footprints:16bars-midjourney-compass, F.Cu at (91.7, 110.8)
- added Ref**: Val**, Footprints:FirstBar, F.Cu at (92.8, 74.2)
- added Ref**: Val**, Footprints:MiddleBar, F.Cu at (92.8, 87.6)
- added Ref**: Val**, Footprints:16Bars-Avant-ModuleTitle-24mm, F.Cu at (91.8, 46.8)
Other:
- board text added: "12"
- board text added: "16"
- board text added: "4"
- board text added: "7"
- board text added: "8"
- board text added: "Bars"
- board text added: "Beats"
- board text added: "Clock"
- board text added: "Last"
- board text added: "Reset"
- board text added: "v3.1"
